File: sketchfan.kicad_sch (KiCad schematic)
At the start: 124 parts, among them SW1 SW_Push, SW10 SW_Push, SW11 SW_Push, SW12 SW_Push, SW13 SW_Push, SW14 SW_Push, SW15 SW_Push, SW16 SW_Push, SW17 SW_Push, SW18 SW_Push, SW19 SW_Push, SW2 SW_Push, SW20 SW_Push, SW21 SW_Push, SW22 SW_Push, SW23 SW_Push, SW24 SW_Push, SW25 SW_Push, SW26 SW_Push, SW27 SW_Push, SW28 SW_Push, SW29 SW_Push, SW3 SW_Push, SW30 SW_Push, SW31 SW_Push, SW32 SW_Push, SW33 SW_Push, SW34 SW_Push, SW35 SW_Push, SW36 SW_Push, SW37 SW_Push, SW38 SW_Push, SW39 SW_Push, SW4 SW_Push, SW40 SW_Push, SW41 SW_Push, SW42 SW_Push, SW43 SW_Push, SW44 SW_Push, SW45 SW_Push, SW46 SW_Push, SW47 SW_Push, SW48 SW_Push, SW49 SW_Push, SW5 SW_Push, SW50 SW_Push, SW51 SW_Push, SW52 SW_Push, SW53 SW_Push, SW54 SW_Push, SW55 SW_Push, SW56 SW_Push, SW57 SW_Push, SW58 SW_Push, SW59 SW_Push, SW6 SW_Push, SW60 SW_Push, SW7 SW_Push, SW8 SW_Push, SW9 SW_Push

Commit message: initial wiring
Connections:
- net col0: now also STM32F401_Board1.28 (A7); no longer STM32F401_Board1.19 (B13)
- net col1: now also STM32F401_Board1.27 (B0); no longer STM32F401_Board1.20 (B12)
- net col10: now also STM32F401_Board1.30 (A5); no longer STM32F401_Board1.33 (A2)
- net col11: now also STM32F401_Board1.29 (A6); no longer STM32F401_Board1.34 (A1)
- net col2: now also STM32F401_Board1.26 (B1); no longer STM32F401_Board1.24 (B10)
- net col3: now also STM32F401_Board1.24 (B10); no longer STM32F401_Board1.26 (B1)
- net col4: now also STM32F401_Board1.20 (B12); no longer STM32F401_Board1.27 (B0)
- net col5: now also STM32F401_Board1.19 (B13); no longer STM32F401_Board1.28 (A7)
- net col6: now also STM32F401_Board1.34 (A1); no longer STM32F401_Board1.29 (A6)
- net col7: now also STM32F401_Board1.33 (A2); no longer STM32F401_Board1.30 (A5)
- net col8: now also STM32F401_Board1.32 (A3); no longer STM32F401_Board1.31 (A4)
- net col9: now also STM32F401_Board1.31 (A4); no longer STM32F401_Board1.32 (A3)
Changed lines of the file:
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@@
+	)
+	(label "col1"
+		(at 86.36 158.75 0)
+		(effects
+			(font
+				(size 1.27 1.27)
+			)
+			(justify left bottom)
+		)
+	)
+	(label "col7"
+		(at 86.36 173.99 0)
+		(effects
+			(font
+				(size 1.27 1.27)
+			)
+			(justify left bottom)
+		)
 	)
 	(label "col1"
@@
 		)
 	)
-	(label "col3"
-		(at 86.36 156.21 0)
-		(effects
-			(font
-				(size 1.27 1.27)
-			)
-			(justify left bottom)
-		)
-	)
 	(label "row3"
 		(at 279.4 106.68 0)
@@
 		)
 	)
-	(label "col6"
-		(at 86.36 163.83 0)
-		(effects
-			(font
-				(size 1.27 1.27)
-			)
-			(justify left bottom)
-		)
-	)
 	(label "row4"
 		(at 55.88 168.91 180)
@@
 		)
 	)
+	(label "col0"
+		(at 86.36 161.29 0)
+		(effects
+			(font
+				(size 1.27 1.27)
+			)
+			(justify left bottom)
+		)
+	)
 	(label "col4"
 		(at 116.84 133.35 0)
@@
 		)
 	)
+	(label "col6"
+		(at 86.36 176.53 0)
+		(effects
+			(font
+				(size 1.27 1.27)
+			)
+			(justify left bottom)
+		)
+	)
 	(label "ENC_R_a"
 		(at 116.84 175.26 180)
@@
 		)
 	)
+	(label "col8"
+		(at 86.3544 171.45 0)
+		(effects
+			(font
+				(size 1.27 1.27)
+			)
+			(justify left bottom)
+		)
+	)
 	(label "ENC_R_push"
 		(at 137.16 175.26 0)
@@
 		)
 	)
-	(label "col5"
-		(at 86.36 161.29 0)
-		(effects
-			(font
-				(size 1.27 1.27)
-			)
-			(justify left bottom)
-		)
-	)
 	(label "ENC_L_push"
 		(at 137.16 153.67 0)
@@
 		)
 	)
+	(label "col4"
+		(at 55.88 143.51 180)
+		(effects
+			(font
+				(size 1.27 1.27)
+			)
+			(justify right bottom)
+		)
+	)
 	(label "col5"
 		(at 135.89 133.35 0)
@@
 		)
 	)
-	(label "col2"
-		(at 86.36 151.13 0)
-		(effects
-			(font
-				(size 1.27 1.27)
-			)
-			(justify left bottom)
-		)
-	)
 	(label "row4"
 		(at 279.4 129.54 0)
@@
 		)
 	)
-	(label "col8"
+	(label "col3"
+		(at 86.36 151.13 0)
+		(effects
+			(font
+				(size 1.27 1.27)
+			)
+			(justify left bottom)
+		)
+	)
+	(label "col9"
 		(at 86.36 168.91 0)
 		(effects
@@
 	)
 	(label "col10"
-		(at 86.36 173.99 0)
+		(at 86.36 166.37 0)
 		(effects
 			(font
@@
 		)
 	)
-	(label "col1"
-		(at 55.88 143.51 180)
-		(effects
-			(font
-				(size 1.27 1.27)
-			)
-			(justify right bottom)
-		)
-	)
-	(label "col0"
-		(at 55.88 146.05 180)
-		(effects
-			(font
-				(size 1.27 1.27)
-			)
-			(justify right bottom)
+	(label "col2"
+		(at 86.36 156.21 0)
+		(effects
+			(font
+				(size 1.27 1.27)
+			)
+			(justify left bottom)
+		)
+	)
+	(label "col11"
+		(at 86.36 163.83 0)
+		(effects
+			(font
+				(size 1.27 1.27)
+			)
+			(justify left bottom)
 		)
 	)
@@
 		)
 	)
-	(label "col4"
-		(at 86.36 158.75 0)
-		(effects
-			(font
-				(size 1.27 1.27)
-			)
-			(justify left bottom)
-		)
-	)
 	(label "col2"
 		(at 78.74 133.35 0)
@@
 		)
 	)
+	(label "col5"
+		(at 55.88 146.05 180)
+		(effects
+			(font
+				(size 1.27 1.27)
+			)
+			(justify right bottom)
+		)
+	)
 	(label "col3"
 		(at 97.79 133.35 0)
@@
 		)
 	)
-	(label "col9"
-		(at 86.36 171.45 0)
-		(effects
-			(font
-				(size 1.27 1.27)
-			)
-			(justify left bottom)
-		)
-	)
-	(label "col7"
-		(at 86.36 166.37 0)
-		(effects
-			(font
-				(size 1.27 1.27)
-			)
-			(justify left bottom)
-		)
-	)
 	(label "col8"
 		(at 218.44 133.35 0)
@@
 		(effects
 			(font
-				(size 1.27 1.27)
-			)
-			(justify left bottom)
-		)
-	)
-	(label "col11"
-		(at 86.36 176.53 0)
-		(effects
-			(font

Commit message: reroute using a better diode footprint and updated via sizes
Parts:
- D1, D10, D11, D12, D13, D14, D15, D16, D17, D18, D19, D2, D20, D21, D22, D23, D24, D25, D26, D27, D28, D29, D3, D30, D31, D32, D33, D34, D35, D36, D37, D38, D39, D4, D40, D41, D42, D43, D44, D45, D46, D47, D48, D49, D5, D50, D51, D52, D53, D54, D55, D56, D57, D58, D59, D6, D60, D7, D8, D9: footprint Diode_THT:D_5W_P5.08mm_Vertical_AnodeUp -> ftvkyo:D_1N4148_TH
Changed lines of the file:
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@@
 			)
 		)
-		(property "Footprint" "Diode_THT:D_5W_P5.08mm_Vertical_AnodeUp"
+		(property "Footprint" "ftvkyo:D_1N4148_TH"
 			(at 82.55 54.61 0)
 			(effects
@@
 			)
 		)
-		(property "Footprint" "Diode_THT:D_5W_P5.08mm_Vertical_AnodeUp"
+		(property "Footprint" "ftvkyo:D_1N4148_TH"
 			(at 203.2 123.19 0)
 			(effects
@@
 			)
 		)
-		(property "Footprint" "Diode_THT:D_5W_P5.08mm_Vertical_AnodeUp"
+		(property "Footprint" "ftvkyo:D_1N4148_TH"
 			(at 203.2 77.47 0)
 			(effects
@@
 			)
 		)
-		(property "Footprint" "Diode_THT:D_5W_P5.08mm_Vertical_AnodeUp"
+		(property "Footprint" "ftvkyo:D_1N4148_TH"
 			(at 165.1 123.19 0)
 			(effects
@@
 			)
 		)
-		(property "Footprint" "Diode_THT:D_5W_P5.08mm_Vertical_AnodeUp"
+		(property "Footprint" "ftvkyo:D_1N4148_TH"
 			(at 120.65 100.33 0)
 			(effects
@@
 			)
 		)
-		(property "Footprint" "Diode_THT:D_5W_P5.08mm_Vertical_AnodeUp"
+		(property "Footprint" "ftvkyo:D_1N4148_TH"
 			(at 222.25 100.33 0)
 			(effects
@@
 			)
 		)
-		(property "Footprint" "Diode_THT:D_5W_P5.08mm_Vertical_AnodeUp"
+		(property "Footprint" "ftvkyo:D_1N4148_TH"
 			(at 241.3 54.61 0)
 			(effects
@@
 			)
 		)
-		(property "Footprint" "Diode_THT:D_5W_P5.08mm_Vertical_AnodeUp"
+		(property "Footprint" "ftvkyo:D_1N4148_TH"
 			(at 82.55 100.33 0)
 			(effects
@@
 			)
 		)
-		(property "Footprint" "Diode_THT:D_5W_P5.08mm_Vertical_AnodeUp"
+		(property "Footprint" "ftvkyo:D_1N4148_TH"
 			(at 260.35 100.33 0)
 			(effects
@@
 			)
 		)
-		(property "Footprint" "Diode_THT:D_5W_P5.08mm_Vertical_AnodeUp"
+		(property "Footprint" "ftvkyo:D_1N4148_TH"
 			(at 120.65 77.47 0)
 			(effects
@@
 			)
 		)
-		(property "Footprint" "Diode_THT:D_5W_P5.08mm_Vertical_AnodeUp"
+		(property "Footprint" "ftvkyo:D_1N4148_TH"
 			(at 260.35 123.19 0)
 			(effects
@@
 			)
 		)
-		(property "Footprint" "Diode_THT:D_5W_P5.08mm_Vertical_AnodeUp"
+		(property "Footprint" "ftvkyo:D_1N4148_TH"
 			(at 63.5 54.61 0)
 			(effects
@@
 			)
 		)
-		(property "Footprint" "Diode_THT:D_5W_P5.08mm_Vertical_AnodeUp"
+		(property "Footprint" "ftvkyo:D_1N4148_TH"
 			(at 101.6 77.47 0)
 			(effects
@@
 			)
 		)
-		(property "Footprint" "Diode_THT:D_5W_P5.08mm_Vertical_AnodeUp"
+		(property "Footprint" "ftvkyo:D_1N4148_TH"
 			(at 120.65 54.61 0)
 			(effects
@@
 			)
 		)
-		(property "Footprint" "Diode_THT:D_5W_P5.08mm_Vertical_AnodeUp"
+		(property "Footprint" "ftvkyo:D_1N4148_TH"
 			(at 184.15 54.61 0)
 			(effects
@@
 			)
 		)
-		(property "Footprint" "Diode_THT:D_5W_P5.08mm_Vertical_AnodeUp"
+		(property "Footprint" "ftvkyo:D_1N4148_TH"
 			(at 101.6 54.61 0)
 			(effects
@@
 			)
 		)
-		(property "Footprint" "Diode_THT:D_5W_P5.08mm_Vertical_AnodeUp"
+		(property "Footprint" "ftvkyo:D_1N4148_TH"
 			(at 82.55 31.75 0)
 			(effects
@@
 			)
 		)
-		(property "Footprint" "Diode_THT:D_5W_P5.08mm_Vertical_AnodeUp"
+		(property "Footprint" "ftvkyo:D_1N4148_TH"
 			(at 184.15 77.47 0)
 			(effects
@@
 			)
 		)
-		(property "Footprint" "Diode_THT:D_5W_P5.08mm_Vertical_AnodeUp"
+		(property "Footprint" "ftvkyo:D_1N4148_TH"
 			(at 25.4 77.47 0)
 			(effects
@@
 			)
 		)
-		(property "Footprint" "Diode_THT:D_5W_P5.08mm_Vertical_AnodeUp"
+		(property "Footprint" "ftvkyo:D_1N4148_TH"
 			(at 101.6 123.19 0)
 			(effects
@@
 			)
 		)
-		(property "Footprint" "Diode_THT:D_5W_P5.08mm_Vertical_AnodeUp"
+		(property "Footprint" "ftvkyo:D_1N4148_TH"
 			(at 260.35 77.47 0)
 			(effects
@@
 			)
 		)
-		(property "Footprint" "Diode_THT:D_5W_P5.08mm_Vertical_AnodeUp"
+		(property "Footprint" "ftvkyo:D_1N4148_TH"
 			(at 101.6 31.75 0)
 			(effects
@@
 			)
 		)
-		(property "Footprint" "Diode_THT:D_5W_P5.08mm_Vertical_AnodeUp"
+		(property "Footprint" "ftvkyo:D_1N4148_TH"
 			(at 25.4 31.75 0)
 			(effects
@@
 			)
 		)
-		(property "Footprint" "Diode_THT:D_5W_P5.08mm_Vertical_AnodeUp"
+		(property "Footprint" "ftvkyo:D_1N4148_TH"
 			(at 63.5 123.19 0)
 			(effects
@@
 			)
 		)
-		(property "Footprint" "Diode_THT:D_5W_P5.08mm_Vertical_AnodeUp"
+		(property "Footprint" "ftvkyo:D_1N4148_TH"
 			(at 222.25 31.75 0)
 			(effects
@@
 			)
 		)
-		(property "Footprint" "Diode_THT:D_5W_P5.08mm_Vertical_AnodeUp"
+		(property "Footprint" "ftvkyo:D_1N4148_TH"
 			(at 260.35 31.75 0)
 			(effects
@@
 			)
 		)
-		(property "Footprint" "Diode_THT:D_5W_P5.08mm_Vertical_AnodeUp"
+		(property "Footprint" "ftvkyo:D_1N4148_TH"
 			(at 165.1 31.75 0)
 			(effects
@@
 			)
 		)
-		(property "Footprint" "Diode_THT:D_5W_P5.08mm_Vertical_AnodeUp"
+		(property "Footprint" "ftvkyo:D_1N4148_TH"
 			(at 82.55 77.47 0)
 			(effects
@@
 			)
 		)
-		(property "Footprint" "Diode_THT:D_5W_P5.08mm_Vertical_AnodeUp"
+		(property "Footprint" "ftvkyo:D_1N4148_TH"
 			(at 44.45 31.75 0)
 			(effects
@@
 			)
 		)
-		(property "Footprint" "Diode_THT:D_5W_P5.08mm_Vertical_AnodeUp"
+		(property "Footprint" "ftvkyo:D_1N4148_TH"
 			(at 44.45 77.47 0)
 			(effects
@@
 			)
 		)
-		(property "Footprint" "Diode_THT:D_5W_P5.08mm_Vertical_AnodeUp"
+		(property "Footprint" "ftvkyo:D_1N4148_TH"
 			(at 241.3 77.47 0)
 			(effects
@@
 			)
 		)
-		(property "Footprint" "Diode_THT:D_5W_P5.08mm_Vertical_AnodeUp"
+		(property "Footprint" "ftvkyo:D_1N4148_TH"
 			(at 241.3 31.75 0)
 			(effects
@@
 			)
 		)
-		(property "Footprint" "Diode_THT:D_5W_P5.08mm_Vertical_AnodeUp"
+		(property "Footprint" "ftvkyo:D_1N4148_TH"
 			(at 63.5 100.33 0)
 			(effects
@@
 			)
 		)
-		(property "Footprint" "Diode_THT:D_5W_P5.08mm_Vertical_AnodeUp"
+		(property "Footprint" "ftvkyo:D_1N4148_TH"
 			(at 25.4 123.19 0)
 			(effects
@@
 			)
 		)
-		(property "Footprint" "Diode_THT:D_5W_P5.08mm_Vertical_AnodeUp"
+		(property "Footprint" "ftvkyo:D_1N4148_TH"
 			(at 44.45 54.61 0)
 			(effects
@@
 			)
 		)
-		(property "Footprint" "Diode_THT:D_5W_P5.08mm_Vertical_AnodeUp"
+		(property "Footprint" "ftvkyo:D_1N4148_TH"
 			(at 120.65 31.75 0)
 			(effects
@@
 			)
 		)
-		(property "Footprint" "Diode_THT:D_5W_P5.08mm_Vertical_AnodeUp"
+		(property "Footprint" "ftvkyo:D_1N4148_TH"
 			(at 184.15 100.33 0)
 			(effects
@@
 			)
 		)
-		(property "Footprint" "Diode_THT:D_5W_P5.08mm_Vertical_AnodeUp"
+		(property "Footprint" "ftvkyo:D_1N4148_TH"
 			(at 120.65 123.19 0)
 			(effects
@@
 			)
 		)
-		(property "Footprint" "Diode_THT:D_5W_P5.08mm_Vertical_AnodeUp"
+		(property "Footprint" "ftvkyo:D_1N4148_TH"
 			(at 44.45 123.19 0)
 			(effects
@@
 			)
 		)
-		(property "Footprint" "Diode_THT:D_5W_P5.08mm_Vertical_AnodeUp"
+		(property "Footprint" "ftvkyo:D_1N4148_TH"
 			(at 165.1 100.33 0)
 			(effects
@@
 			)
 		)
-		(property "Footprint" "Diode_THT:D_5W_P5.08mm_Vertical_AnodeUp"
+		(property "Footprint" "ftvkyo:D_1N4148_TH"
 			(at 222.25 54.61 0)
 			(effects
@@
 			)
 		)
-		(property "Footprint" "Diode_THT:D_5W_P5.08mm_Vertical_AnodeUp"
+		(property "Footprint" "ftvkyo:D_1N4148_TH"
 			(at 184.15 31.75 0)
 			(effects
@@
 			)
 		)
-		(property "Footprint" "Diode_THT:D_5W_P5.08mm_Vertical_AnodeUp"
+		(property "Footprint" "ftvkyo:D_1N4148_TH"
 			(at 25.4 100.33 0)
 			(effects
@@
 			)
 		)
-		(property "Footprint" "Diode_THT:D_5W_P5.08mm_Vertical_AnodeUp"
+		(property "Footprint" "ftvkyo:D_1N4148_TH"
 			(at 101.6 100.33 0)
 			(effects
@@
 			)
 		)
-		(property "Footprint" "Diode_THT:D_5W_P5.08mm_Vertical_AnodeUp"
+		(property "Footprint" "ftvkyo:D_1N4148_TH"
 			(at 165.1 54.61 0)
 			(effects
@@
 			)
 		)
-		(property "Footprint" "Diode_THT:D_5W_P5.08mm_Vertical_AnodeUp"
+		(property "Footprint" "ftvkyo:D_1N4148_TH"
 			(at 203.2 31.75 0)
 			(effects
@@
 			)
 		)
-		(property "Footprint" "Diode_THT:D_5W_P5.08mm_Vertical_AnodeUp"
+		(property "Footprint" "ftvkyo:D_1N4148_TH"
 			(at 165.1 77.47 0)
 			(effects
@@
 			)
 		)
-		(property "Footprint" "Diode_THT:D_5W_P5.08mm_Vertical_AnodeUp"
+		(property "Footprint" "ftvkyo:D_1N4148_TH"
 			(at 203.2 54.61 0)
 			(effects
@@
 			)
 		)
-		(property "Footprint" "Diode_THT:D_5W_P5.08mm_Vertical_AnodeUp"
+		(property "Footprint" "ftvkyo:D_1N4148_TH"
 			(at 241.3 123.19 0)
 			(effects
@@
 			)
 		)
-		(property "Footprint" "Diode_THT:D_5W_P5.08mm_Vertical_AnodeUp"
+		(property "Footprint" "ftvkyo:D_1N4148_TH"
 			(at 44.45 100.33 0)
 			(effects
@@
 			)
 		)
-		(property "Footprint" "Diode_THT:D_5W_P5.08mm_Vertical_AnodeUp"
+		(property "Footprint" "ftvkyo:D_1N4148_TH"
 			(at 63.5 31.75 0)
 			(effects
@@
 			)
 		)
-		(property "Footprint" "Diode_THT:D_5W_P5.08mm_Vertical_AnodeUp"
+		(property "Footprint" "ftvkyo:D_1N4148_TH"
 			(at 82.55 123.19 0)
 			(effects
@@
 			)
 		)
-		(property "Footprint" "Diode_THT:D_5W_P5.08mm_Vertical_AnodeUp"
+		(property "Footprint" "ftvkyo:D_1N4148_TH"
 			(at 222.25 123.19 0)
 			(effects
@@
 			)
 		)
-		(property "Footprint" "Diode_THT:D_5W_P5.08mm_Vertical_AnodeUp"
+		(property "Footprint" "ftvkyo:D_1N4148_TH"
 			(at 222.25 77.47 0)
 			(effects
@@
 			)
 		)
-		(property "Footprint" "Diode_THT:D_5W_P5.08mm_Vertical_AnodeUp"
+		(property "Footprint" "ftvkyo:D_1N4148_TH"
 			(at 260.35 54.61 0)
 			(effects
@@
 			)
 		)
-		(property "Footprint" "Diode_THT:D_5W_P5.08mm_Vertical_AnodeUp"
+		(property "Footprint" "ftvkyo:D_1N4148_TH"
 			(at 63.5 77.47 0)
 			(effects
@@
 			)
 		)
-		(property "Footprint" "Diode_THT:D_5W_P5.08mm_Vertical_AnodeUp"
+		(property "Footprint" "ftvkyo:D_1N4148_TH"
 			(at 241.3 100.33 0)
 			(effects
@@
 			)
 		)
-		(property "Footprint" "Diode_THT:D_5W_P5.08mm_Vertical_AnodeUp"
+		(property "Footprint" "ftvkyo:D_1N4148_TH"
 			(at 203.2 100.33 0)
 			(effects
@@
 			)
 		)
-		(property "Footprint" "Diode_THT:D_5W_P5.08mm_Vertical_AnodeUp"
+		(property "Footprint" "ftvkyo:D_1N4148_TH"
 			(at 25.4 54.61 0)
 			(effects
@@
 			)
 		)
-		(property "Footprint" "Diode_THT:D_5W_P5.08mm_Vertical_AnodeUp"
+		(property "Footprint" "ftvkyo:D_1N4148_TH"
 			(at 184.15 123.19 0)
 			(effects
