File: sketchfan.kicad_pcb (KiCad board)
At the start: 2 copper layers, 124 parts, among them SW1 SW_Push, SW10 SW_Push, SW11 SW_Push, SW12 SW_Push, SW13 SW_Push, SW14 SW_Push, SW15 SW_Push, SW16 SW_Push, SW17 SW_Push, SW18 SW_Push, SW19 SW_Push, SW2 SW_Push, SW20 SW_Push, SW21 SW_Push, SW22 SW_Push, SW23 SW_Push, SW24 SW_Push, SW25 SW_Push, SW26 SW_Push, SW27 SW_Push, SW28 SW_Push, SW29 SW_Push, SW3 SW_Push, SW30 SW_Push, SW31 SW_Push, SW32 SW_Push, SW33 SW_Push, SW34 SW_Push, SW35 SW_Push, SW36 SW_Push, SW37 SW_Push, SW38 SW_Push, SW39 SW_Push, SW4 SW_Push, SW40 SW_Push, SW41 SW_Push, SW42 SW_Push, SW43 SW_Push, SW44 SW_Push, SW45 SW_Push, SW46 SW_Push, SW47 SW_Push, SW48 SW_Push, SW49 SW_Push, SW5 SW_Push, SW50 SW_Push, SW51 SW_Push, SW52 SW_Push, SW53 SW_Push, SW54 SW_Push, SW55 SW_Push, SW56 SW_Push, SW57 SW_Push, SW58 SW_Push, SW59 SW_Push, SW6 SW_Push, SW60 SW_Push, SW7 SW_Push, SW8 SW_Push, SW9 SW_Push

Commit message: initial wiring
Parts:
- moved D1 19.1 mm to (-40.4, -53.7), turned to -105 degrees
- moved D7 19.0 mm to (-44.9, -36.2), turned to -105 degrees
- moved D13 18.8 mm to (-49.9, -18.7), turned to -105 degrees
- moved D20 0.69 mm to (-36.1, 3.74)
- moved D25 0.24 mm to (-22.1, 23.7)
- moved D19 0.11 mm to (-41.1, 21.7)
Connections:
- STM32F401_Board1 pad 19: /col0 -> /col5
- STM32F401_Board1 pad 20: /col1 -> /col4
- STM32F401_Board1 pad 24: /col2 -> /col3
- STM32F401_Board1 pad 26: /col3 -> /col2
- STM32F401_Board1 pad 27: /col4 -> /col1
- STM32F401_Board1 pad 28: /col5 -> /col0
- STM32F401_Board1 pad 29: /col6 -> /col11
- STM32F401_Board1 pad 30: /col7 -> /col10
- STM32F401_Board1 pad 31: /col8 -> /col9
- STM32F401_Board1 pad 32: /col9 -> /col8
- STM32F401_Board1 pad 33: /col10 -> /col7
- STM32F401_Board1 pad 34: /col11 -> /col6
Routing:
- net /row2: track 0.00 -> 439.9 mm, vias 0 -> 26
- net /row3: track 0.00 -> 408.2 mm, vias 1 -> 20
- net /row0: track 0.00 -> 383.1 mm, vias 0 -> 24
- net /row1: track 0.00 -> 382.6 mm, vias 0 -> 24
- net /row4: track 0.00 -> 329.8 mm, vias 0 -> 2
- net /col0: track 0.00 -> 316.7 mm
- net /col1: track 0.00 -> 314.5 mm
- net /col11: track 0.00 -> 297.1 mm
- net /col2: track 0.00 -> 239.4 mm
- net /col10: track 0.00 -> 235.7 mm
- net /col9: track 0.00 -> 221.8 mm
- net /col3: track 0.00 -> 212.6 mm
- net /col8: track 0.00 -> 209.6 mm
- net GND: track 0.00 -> 199.8 mm, vias 0 -> 2
- net /col7: track 0.00 -> 191.5 mm
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
Commit message: neat wiring
Routing:
- net /col1: track 314.5 -> 295.2 mm
- net /col11: track 297.1 -> 282.3 mm
- net /row0: track 383.1 -> 369.0 mm, vias 24 -> 22
- net /col10: track 235.7 -> 223.9 mm
- net /col8: track 209.6 -> 198.1 mm
- net /col9: track 221.8 -> 210.8 mm
- net /col0: track 316.7 -> 305.8 mm
- net /col7: track 191.5 -> 181.4 mm
- net /col6: track 175.0 -> 166.6 mm
- net /col3: track 212.6 -> 208.8 mm
- net /col2: track 239.4 -> 236.6 mm
- net /row3: track 408.2 -> 406.2 mm
- net /row4: track 329.8 -> 331.6 mm
- net GND: track 199.8 -> 198.5 mm
- net /buzz: track 68.6 -> 69.9 mm
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
Commit message: add simple edge cuts
Routing:
- net /row4: track 331.6 -> 330.5 mm
Other:
- board outline added: 302 x 137.4 mm

Commit message: reduce width to fit in 300mm
Other:
- board size 302 x 137.4 mm -> 300 x 137.4 mm
Changed lines of the file:
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@@
+	)
+	(gr_line
+		(start -36 -68)
+		(end 15 -64.5)
+		(stroke
+			(width 0.05)
+			(type default)
+		)
+		(layer "Edge.Cuts")
+	)
+	(gr_line
+		(start 13 42)
+		(end -62 22)
+		(stroke
+			(width 0.05)
+			(type default)
+		)
+		(layer "Edge.Cuts")
 	)
 	(gr_line
 		(start 47 56)
 		(end 31 47)
-		(stroke
-			(width 0.05)
-			(type default)
-		)
-		(layer "Edge.Cuts")
-	)
-	(gr_line
-		(start 133 -64)
-		(end 84 -48)
-		(stroke
-			(width 0.05)
-			(type default)
-		)
-		(layer "Edge.Cuts")
-	)
-	(gr_line
-		(start 63 69)
-		(end 47 56)
 		(stroke
 			(width 0.05)
@@
 	)
 	(gr_line
-		(start 13 42)
-		(end -62 22)
-		(stroke
-			(width 0.05)
-			(type default)
-		)
-		(layer "Edge.Cuts")
-	)
-	(gr_line
-		(start -63 -56)
-		(end -36 -68)
-		(stroke
-			(width 0.05)
-			(type default)
-		)
-		(layer "Edge.Cuts")
-	)
-	(gr_line
-		(start -77 -4)
-		(end -63 -56)
+		(start 15 -64.5)
+		(end 64 -48)
 		(stroke
 			(width 0.05)
@@
 	)
 	(gr_line
-		(start 31 47)
-		(end 13 42)
-		(stroke
-			(width 0.05)
-			(type default)
-		)
-		(layer "Edge.Cuts")
-	)
-	(gr_line
-		(start 225 -4)
-		(end 211 -56)
+		(start 224 -4)
+		(end 210 -56)
+		(stroke
+			(width 0.05)
+			(type default)
+		)
+		(layer "Edge.Cuts")
+	)
+	(gr_line
+		(start 63 69)
+		(end 47 56)
 		(stroke
 			(width 0.05)
@@
 	)
 	(gr_line
-		(start 225 -4)
+		(start 224 -4)
 		(end 210 22)
-		(stroke
-			(width 0.05)
-			(type default)
-		)
-		(layer "Edge.Cuts")
-	)
-	(gr_line
-		(start 15 -64)
-		(end 64 -48)
-		(stroke
-			(width 0.05)
-			(type default)
-		)
-		(layer "Edge.Cuts")
-	)
-	(gr_line
-		(start -36 -68)
-		(end 15 -64)
 		(stroke
 			(width 0.05)
@@
 	)
 	(gr_line
+		(start -76 -4)
+		(end -62 22)
+		(stroke
+			(width 0.05)
+			(type default)
+		)
+		(layer "Edge.Cuts")
+	)
+	(gr_line
+		(start 133 -64.5)
+		(end 84 -48)
+		(stroke
+			(width 0.05)
+			(type default)
+		)
+		(layer "Edge.Cuts")
+	)
+	(gr_line
+		(start -62 -56)
+		(end -36 -68)
+		(stroke
+			(width 0.05)
+			(type default)
+		)
+		(layer "Edge.Cuts")
+	)
+	(gr_line
 		(start 84 -48)
 		(end 64 -48)
@@
 	)
 	(gr_line
-		(start 211 -56)
+		(start 210 -56)
 		(end 184 -68)
 		(stroke
@@
 	)
 	(gr_line
-		(start -77 -4)
-		(end -62 22)
-		(stroke
-			(width 0.05)
-			(type default)
-		)
-		(layer "Edge.Cuts")
-	)
-	(gr_line
 		(start 184 -68)
-		(end 133 -64)
+		(end 133 -64.5)
+		(stroke
+			(width 0.05)
+			(type default)
+		)
+		(layer "Edge.Cuts")
+	)
+	(gr_line
+		(start 31 47)
+		(end 13 42)
 		(stroke
 			(width 0.05)
@@
 		(stroke
 			(width 0.05)
+			(type default)
+		)
+		(layer "Edge.Cuts")
+	)
+	(gr_line
+		(start -76 -4)
+		(end -62 -56)
+		(stroke
+			(width 0.05)

Commit message: reroute using a better diode footprint and updated via sizes
Parts:
- D1, D10, D11, D12, D13, D14, D15, D16, D17, D18, D19, D2, D20, D21, D22, D23, D24, D25, D26, D27, D28, D29, D3, D30, D31, D32, D33, D34, D35, D36, D37, D38, D39, D4, D40, D41, D42, D43, D44, D45, D46, D47, D48, D49, D5, D50, D51, D52, D53, D54, D55, D56, D57, D58, D59, D6, D60, D7, D8, D9: footprint Diode_THT:D_5W_P5.08mm_Vertical_AnodeUp -> ftvkyo:D_1N4148_TH; moved to F.Cu
- moved D55 20.0 mm to (96.0, 48.9), turned to 40 degrees
- moved D56 19.3 mm to (113.3, 38.9), turned to 30 degrees
- moved D7 15.4 mm to (-49.0, -21.4), turned to -15 degrees
- moved D1 15.4 mm to (-44.4, -38.9), turned to -15 degrees
- moved D13 15.3 mm to (-53.8, -3.97), turned to -15 degrees
- moved D2 3.71 mm to (-21.3, -51.3), turned to -15 degrees
- moved D8 3.69 mm to (-26.0, -33.9), turned to -15 degrees
- moved D14 3.68 mm to (-30.7, -16.5), turned to -15 degrees
- moved D3 3.66 mm to (-2.27, -49.3), turned to -15 degrees
- moved D12 3.66 mm to (47.5, -14.2), turned to -15 degrees
- moved D4 3.66 mm to (16.9, -47.3), turned to -15 degrees
- moved D58 3.62 mm to (150.6, 25.2), turned to 15 degrees
- moved D26 3.62 mm to (-1.81, 22.3), turned to -15 degrees
- moved D28 3.62 mm to (33.4, 38.0), turned to -15 degrees
- moved D23 3.62 mm to (20.4, 12.7), turned to -15 degrees
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Routing:
- net /col1: track 295.2 -> 258.6 mm
- net /row0: track 369.0 -> 400.8 mm
- net /row1: track 382.9 -> 414.7 mm
- net /row2: track 438.8 -> 469.3 mm
- net /col0: track 305.8 -> 280.0 mm, vias 0 -> 2
- net /row3: track 406.2 -> 427.8 mm
- net Net-(D55-A): track 24.5 -> 3.85 mm
- net Net-(D56-A): track 23.3 -> 3.77 mm
- net /col7: track 181.4 -> 188.3 mm
- net /row4: track 330.5 -> 323.8 mm
- net /col6: track 166.6 -> 172.3 mm
- net /col11: track 282.3 -> 278.2 mm
- net /col9: track 210.8 -> 207.6 mm
- net /col8: track 198.1 -> 200.7 mm
- net /col2: track 236.6 -> 234.9 mm
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
Commit message: move the PCB to be in positive coordinates
Parts:
- moved D32 103.5 mm to (209.3, 24.5)
- moved D42 103.5 mm to (292.9, 42.6)
- moved D45 103.5 mm to (236.2, 51.5)
- moved D53 103.5 mm to (279.1, 64.9)
- moved D55 103.5 mm to (173.4, 117.7)
- moved D56 103.5 mm to (190.6, 107.6)
- moved D7 103.5 mm to (28.3, 47.4)
- moved SW31 103.5 mm to (181.9, 32.5)
- moved SW40 103.5 mm to (240.8, 32.2)
- moved SW51 103.5 mm to (231.0, 69.0)
- moved SW53 103.5 mm to (269.2, 64.9)
- moved BZ1 103.5 mm to (151.3, 97.8)
- moved D11 103.5 mm to (107.1, 46.8)
- moved D14 103.5 mm to (46.6, 52.2)
- moved D19 103.5 mm to (37.3, 87.2)
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